Commit message: Updated rover and added gazebo plugins

File: description/rover_core.xacro (robot description, xacro)
@@ -10,5 +10,5 @@
         <parent link="base_link"/>
         <child link="chassis"/>
-        <origin xyz="0 0 0"/>
+        <origin xyz="1 0 1"/>
     </joint>
     <link name="chassis">
@@ -30,9 +30,12 @@
         </xacro:inertial_box>
     </link>
+    <gazebo reference="chassis">
+        <material>Gazebo/Black</material>
+    </gazebo>
     <!-- Suspension-->
     <!-- WHEELS -->
     <!-- Left Front -->
     <joint name="left_front_wheel_joint" type="continuous">
-        <parent link="base_link"/>
+        <parent link="chassis"/>
         <child link="left_front_wheel"/>
         <origin xyz="0.155 0.15 -.15" rpy="-${pi/2} 0 0"/>
@@ -55,7 +58,10 @@
         </xacro:inertial_cylinder>
     </link>
+    <gazebo reference="left_front_wheel">
+        <material>Gazebo/White</material>
+    </gazebo>
     <!-- Left Back -->
     <joint name="left_back_wheel_joint" type="continuous">
-        <parent link="base_link"/>
+        <parent link="chassis"/>
         <child link="left_back_wheel"/>
         <origin xyz="-0.155 0.15 -.15" rpy="-${pi/2} 0 0"/>
@@ -78,7 +84,10 @@
         </xacro:inertial_cylinder>
     </link>
+    <gazebo reference="left_back_wheel">
+        <material>Gazebo/White</material>
+    </gazebo>
     <!-- Right Front -->
     <joint name="right_front_wheel_joint" type="continuous">
-        <parent link="base_link"/>
+        <parent link="chassis"/>
         <child link="right_front_wheel"/>
         <origin xyz="0.155 -0.15 -.15" rpy="${pi/2} 0 0"/>
@@ -101,7 +110,10 @@
         </xacro:inertial_cylinder>
     </link>
+    <gazebo reference="right_front_wheel">
+        <material>Gazebo/White</material>
+    </gazebo>
     <!-- Right Back -->
     <joint name="right_back_wheel_joint" type="continuous">
-        <parent link="base_link"/>
+        <parent link="chassis"/>
         <child link="right_back_wheel"/>
         <origin xyz="-0.155 -0.15 -.15" rpy="${pi/2} 0 0"/>
@@ -124,3 +136,6 @@
         </xacro:inertial_cylinder>
     </link>
+    <gazebo reference="right_back_wheel">
+        <material>Gazebo/White</material>
+    </gazebo>
 </robot>

File: description/rover_main.urdf.xacro (robot description, xacro)
@@ -2,3 +2,6 @@
 <robot xmlns:xacro="http://www.ros.org/wiki/xacro" name="robot">
     <xacro:include filename="rover_core.xacro" />
+    <xacro:include filename="ros2_control.xacro"/>
+    <xacro:include filename="lidar.xacro"/>
+    <xacro:include filename="cam.xacro"/>
 </robot>
