Commit message: Updated sensor config

File: description/cam.xacro (robot description, xacro)
@@ -1,10 +1,15 @@
 <?xml version="1.0"?>
 <robot xmlns:xacro="http://www.ros.org/wiki/xacro" name="robot">
-    <joint name="cam_joint" type="fixed">
+    <joint name="front_cam_joint" type="fixed">
         <parent link="chassis"/>
-        <child link="cam_frame"/>
+        <child link="front_cam_frame"/>
         <origin xyz="0.25 0 0.02" rpy="0 0 0"/>
     </joint>
-    <link name="cam_frame">
+    <joint name="rear_cam_joint" type="fixed">
+        <parent link="chassis"/>
+        <child link="rear_cam_frame"/>
+        <origin xyz="-0.25 0 0.02" rpy="0 0 0"/>
+    </joint>
+    <link name="front_cam_frame">
         <visual>
             <origin xyz="0 0 0"/>
@@ -24,13 +29,37 @@
         </xacro:inertial_box>
     </link>
-    <joint name="camera_optical_joint" type="fixed">
-        <origin xyz="0 0 0" rpy="${-pi/2} 0 ${-pi/2}" />
-        <parent link="cam_frame" />
-        <child link="camera_link_optical" />
+    <link name="rear_cam_frame">
+        <visual>
+            <origin xyz="0 0 0"/>
+            <geometry>
+                <box size="0.001 0.1 0.01"/>
+            </geometry>
+            <material name="orange"/>
+        </visual>
+        <collision>
+            <origin xyz="0 0 0"/>
+            <geometry>
+                <box size="0.001 0.1 0.01"/>
+            </geometry>
+        </collision>
+        <xacro:inertial_box mass="0.1" x="0.001" y="0.1" z="0.01">
+            <origin xyz="0 0 0" rpy="0 0 0"/>
+        </xacro:inertial_box>
+    </link>
+    <joint name="front_camera_optical_joint" type="fixed">
+        <origin xyz="0 0 0" rpy="0 0 0" />
+        <parent link="front_cam_frame" />
+        <child link="front_camera_link_optical" />
     </joint>
-    <link name="camera_link_optical"></link>
-    <gazebo reference="cam_frame">
+    <joint name="rear_camera_optical_joint" type="fixed">
+        <origin xyz="0 0 0" rpy="0 0 ${-pi}" />
+        <parent link="rear_cam_frame" />
+        <child link="rear_camera_link_optical" />
+    </joint>
+    <link name="front_camera_link_optical"></link>
+    <link name="rear_camera_link_optical"></link>
+    <gazebo reference="front_camera_link_optical">
         <material>Gazebo/Orange</material>
-        <sensor name="camera" type="camera">
+        <sensor name="front_camera" type="camera">
             <pose> 0 0 0 0 0 0 </pose>
             <visualize>true</visualize>
@@ -40,6 +69,6 @@
                 <image>
                     <format>R8G8B8</format>
-                    <width>640</width>
-                    <height>480</height>
+                    <width>1280</width>
+                    <height>720</height>
                 </image>
                 <clip>
@@ -48,6 +77,29 @@
                 </clip>
             </camera>
-            <plugin name="camera_controller" filename="libgazebo_ros_camera.so">
-                <frame_name>camera_link_optical</frame_name>
+            <plugin name="front_camera_controller" filename="libgazebo_ros_camera.so">
+                <frame_name>front_camera_link_optical</frame_name>
+            </plugin>
+        </sensor>
+    </gazebo>
+    <gazebo reference="rear_camera_link_optical">
+        <material>Gazebo/Orange</material>
+        <sensor name="rear_camera" type="camera">
+            <pose> 0 0 0 0 0 0 </pose>
+            <visualize>true</visualize>
+            <update_rate>10</update_rate>
+            <camera>
+                <horizontal_fov>1.089</horizontal_fov>
+                <image>
+                    <format>R8G8B8</format>
+                    <width>1280</width>
+                    <height>720</height>
+                </image>
+                <clip>
+                    <near>0.05</near>
+                    <far>8.0</far>
+                </clip>
+            </camera>
+            <plugin name="rear_camera_controller" filename="libgazebo_ros_camera.so">
+                <frame_name>rear_camera_link_optical</frame_name>
             </plugin>
         </sensor>

File: description/lidar.xacro (robot description, xacro)
@@ -1,10 +1,15 @@
 <?xml version="1.0"?>
 <robot xmlns:xacro="http://www.ros.org/wiki/xacro" name="robot">
-    <joint name="lidar_joint" type="fixed">
+    <joint name="front_lidar_joint" type="fixed">
         <parent link="chassis"/>
-        <child link="lidar_frame"/>
+        <child link="front_lidar_frame"/>
         <origin xyz="0.25 0 -0.02" rpy="0 0 0"/>
     </joint>
-    <link name="lidar_frame">
+    <joint name="rear_lidar_joint" type="fixed">
+        <parent link="chassis"/>
+        <child link="rear_lidar_frame"/>
+        <origin xyz="-0.25 0 -0.02" rpy="0 0 ${-pi}"/>
+    </joint>
+    <link name="front_lidar_frame">
         <visual>
             <origin xyz="0 0 0"/>
@@ -24,19 +29,44 @@
         </xacro:inertial_box>
     </link>
-    <joint name="lidar_optical_joint" type="fixed">
+    <link name="rear_lidar_frame">
+        <visual>
+            <origin xyz="0 0 0"/>
+            <geometry>
+                <box size="0.001 0.1 0.01"/>
+            </geometry>
+            <material name="blue"/>
+        </visual>
+        <collision>
+            <origin xyz="0 0 0"/>
+            <geometry>
+                <box size="0.5 0.3 0.2"/>
+            </geometry>
+        </collision>
+        <xacro:inertial_box mass="0.1" x="0.001" y="0.1" z="0.01">
+            <origin xyz="0 0 0" rpy="0 0 0"/>
+        </xacro:inertial_box>
+    </link>
+    <joint name="front_lidar_optical_joint" type="fixed">
         <origin xyz="0 0 0" rpy="${-pi/2} 0 ${-pi/2}" />
-        <parent link="lidar_frame" />
-        <child link="lidar_link_optical" />
+        <parent link="front_lidar_frame" />
+        <child link="front_lidar_link_optical" />
     </joint>
-    <link name="lidar_link_optical"></link>
-    <gazebo reference="lidar_frame">
+    <joint name="rear_lidar_optical_joint" type="fixed">
+        <origin xyz="0 0 0" rpy="${-pi/2} 0 ${-pi/2}" />
+        <parent link="rear_lidar_frame" />
+        <child link="rear_lidar_link_optical" />
+    </joint>
+    <link name="front_lidar_link_optical"></link>
+    <link name="rear_lidar_link_optical"></link>
+    <gazebo reference="front_lidar_frame">
         <material>Gazebo/Blue</material>
-        <sensor name="lidar" type="depth">
+        <sensor name="front_lidar" type="depth">
+            <pose> 0 0 0 0 0 0 </pose>
             <update_rate>20</update_rate>
             <camera>
                 <horizontal_fov>1.047198</horizontal_fov>
                 <image>
-                    <width>640</width>
-                    <height>480</height>
+                    <width>224</width>
+                    <height>172</height>
                     <format>R8G8B8</format>
                 </image>
@@ -46,6 +76,28 @@
                 </clip>
             </camera>
-            <plugin name="lidar_controller" filename="libgazebo_ros_camera.so">
-                <frame_name>lidar_link_optical</frame_name>
+            <plugin name="front_lidar_controller" filename="libgazebo_ros_camera.so">
+                <frame_name>front_lidar_link_optical</frame_name>
+            </plugin>
+        </sensor>
+    </gazebo>
+    <gazebo reference="rear_lidar_frame">
+        <material>Gazebo/Blue</material>
+        <sensor name="rear_lidar" type="depth">
+            <pose> 0 0 0 0 0 0 </pose>
+            <update_rate>20</update_rate>
+            <camera>
+                <horizontal_fov>1.047198</horizontal_fov>
+                <image>
+                    <width>224</width>
+                    <height>172</height>
+                    <format>R8G8B8</format>
+                </image>
+                <clip>
+                    <near>0.05</near>
+                    <far>20</far>
+                </clip>
+            </camera>
+            <plugin name="rear_lidar_controller" filename="libgazebo_ros_camera.so">
+                <frame_name>rear_lidar_link_optical</frame_name>
             </plugin>
         </sensor>
